File: modular_software_configurable_io_plc/modular_software_configurable_io_plc.kicad_sch (KiCad schematic)
At the start: 35 parts, among them J1 FW-14-03-G-D-085-155, J10 CLP-108-02-G-D-BE, J11 CLP-102-02-G-D-BE, J12 CLP-102-02-G-D-BE, J13 CLP-102-02-G-D-BE, J14 CLP-108-02-G-D-BE, J15 FW-14-03-G-D-085-155, J16 FW-02-03-G-D-085-155, J17 FW-02-03-G-D-085-155, J18 FW-02-03-G-D-085-155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

Commit message: Backup
Parts:
- J19: footprint connector_footprints:FW-02-03-G-D-085-155 -> connector_footprints:FW-03-03-G-D-085-155; symbol UNITED_CONNECTORS_DATA_BASE:J_FW-02-03-G-D-085-155 -> UNITED_CONNECTORS_DATA_BASE:J_FW-03-03-G-D-085-155; MPN FW-02-03-G-D-085-155 -> FW-03-03-G-D-085-155; Pin Count 2 -> 3; Symbol Name J_FW-02-03-G-D-085-155 -> J_FW-03-03-G-D-085-155; Trustedparts Search https://www.trustedparts.com/en/search/FW-02-03-G-D-085-155 -> https://www.trustedparts.com/en/search/FW-03-03-G-D-085-155
Changed lines of the file:
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@@
 	)
 	(symbol
-		(lib_id "UNITED_CONNECTORS_DATA_BASE:J_FW-02-03-G-D-085-155")
+		(lib_id "UNITED_CONNECTORS_DATA_BASE:J_FW-03-03-G-D-085-155")
 		(at 251.46 55.88 0)
 		(unit 1)
@@
 		(fields_autoplaced yes)
 		(property "Reference" "J19"
-			(at 251.46 46.99 0)
+			(at 251.46 45.72 0)
 			(effects
 				(font
@@
 		)
 		(property "Value" "FW-02-03-G-D-085-155"
-			(at 251.46 49.53 0)
-			(effects
-				(font
-					(size 1.27 1.27)
-				)
-			)
-		)
-		(property "Footprint" "connector_footprints:FW-02-03-G-D-085-155"
-			(at 256.54 63.5 0)
+			(at 251.46 48.26 0)
+			(effects
+				(font
+					(size 1.27 1.27)
+				)
+			)
+		)
+		(property "Footprint" "connector_footprints:FW-03-03-G-D-085-155"
+			(at 256.54 64.77 0)
 			(show_name yes)
 			(effects
@@
 		)
 		(property "Datasheet" "https://suddendocs.samtec.com/catalog_english/fw_sm.pdf?_gl=1*1xtxv9c*_gcl_au*MTM0MTYyNTQ5MS4xNzM2MDk5MTUz*_ga*MTYxNDYyMTQ0Mi4xNzM2MDk5MTUz*_ga_3KFNZC07WW*MTczODE2NTI0NS4zMi4xLjE3MzgxNjU1NjMuNjAuMC4w"
-			(at 256.54 66.04 0)
-			(show_name yes)
-			(effects
-				(font
-					(size 1.27 1.27)
-				)
-				(justify left)
-				(hide yes)
-			)
-		)
-		(property "Description" "Samtec FW-xx-03-G-D-085-155 series,  2 positions connector,  1.27 mm pitch,  Black,  Vertical mounting,  5.2 A,  300 V,  Surface Mount,  Gold plated"
-			(at 256.54 68.58 0)
+			(at 256.54 67.31 0)
+			(show_name yes)
+			(effects
+				(font
+					(size 1.27 1.27)
+				)
+				(justify left)
+				(hide yes)
+			)
+		)
+		(property "Description" "Samtec FW-xx-03-G-D-085-155 series,  3 positions connector,  1.27 mm pitch,  Black,  Vertical mounting,  5.2 A,  300 V,  Surface Mount,  Gold plated"
+			(at 256.54 69.85 0)
 			(show_name yes)
 			(effects
@@
 		)
 		(property "Color" "Black"
-			(at 256.54 71.12 0)
+			(at 256.54 72.39 0)
 			(show_name yes)
 			(effects
@@
 		)
 		(property "Contact Plating" "Gold"
-			(at 256.54 73.66 0)
+			(at 256.54 74.93 0)
 			(show_name yes)
 			(effects
@@
 		)
 		(property "Current Rating (A)" "5.2"
-			(at 256.54 76.2 0)
-			(show_name yes)
-			(effects
-				(font
-					(size 1.27 1.27)
-				)
-				(justify left)
-				(hide yes)
-			)
-		)
-		(property "MPN" "FW-02-03-G-D-085-155"
-			(at 256.54 78.74 0)
+			(at 256.54 77.47 0)
+			(show_name yes)
+			(effects
+				(font
+					(size 1.27 1.27)
+				)
+				(justify left)
+				(hide yes)
+			)
+		)
+		(property "MPN" "FW-03-03-G-D-085-155"
+			(at 256.54 80.01 0)
 			(show_name yes)
 			(effects
@@
 		)
 		(property "Manufacturer" "Samtec"
-			(at 256.54 81.28 0)
+			(at 256.54 82.55 0)
 			(show_name yes)
 			(effects
@@
 		)
 		(property "Mounting Angle" "Vertical"
-			(at 256.54 83.82 0)
+			(at 256.54 85.09 0)
 			(show_name yes)
 			(effects
@@
 		)
 		(property "Mounting Style" "Surface Mount"
-			(at 256.54 86.36 0)
+			(at 256.54 87.63 0)
 			(show_name yes)
 			(effects
@@
 		)
 		(property "Number of Rows" "2"
-			(at 256.54 88.9 0)
-			(show_name yes)
-			(effects
-				(font
-					(size 1.27 1.27)
-				)
-				(justify left)
-				(hide yes)
-			)
-		)
-		(property "Pin Count" "2"
-			(at 256.54 91.44 0)
+			(at 256.54 90.17 0)
+			(show_name yes)
+			(effects
+				(font
+					(size 1.27 1.27)
+				)
+				(justify left)
+				(hide yes)
+			)
+		)
+		(property "Pin Count" "3"
+			(at 256.54 92.71 0)
 			(show_name yes)
 			(effects
@@
 		)
 		(property "Pitch (mm)" "1.27"
-			(at 256.54 93.98 0)
+			(at 256.54 95.25 0)
 			(show_name yes)
 			(effects
@@
 		)
 		(property "Series" "FW-xx-03-G-D-085-155"
-			(at 256.54 96.52 0)
-			(show_name yes)
-			(effects
-				(font
-					(size 1.27 1.27)
-				)
-				(justify left)
-				(hide yes)
-			)
-		)
-		(property "Symbol Name" "J_FW-02-03-G-D-085-155"
-			(at 256.54 99.06 0)
-			(show_name yes)
-			(effects
-				(font
-					(size 1.27 1.27)
-				)
-				(justify left)
-				(hide yes)
-			)
-		)
-		(property "Trustedparts Search" "https://www.trustedparts.com/en/search/FW-02-03-G-D-085-155"
-			(at 256.54 101.6 0)
+			(at 256.54 97.79 0)
+			(show_name yes)
+			(effects
+				(font
+					(size 1.27 1.27)
+				)
+				(justify left)
+				(hide yes)
+			)
+		)
+		(property "Symbol Name" "J_FW-03-03-G-D-085-155"
+			(at 256.54 100.33 0)
+			(show_name yes)
+			(effects
+				(font
+					(size 1.27 1.27)
+				)
+				(justify left)
+				(hide yes)
+			)
+		)
+		(property "Trustedparts Search" "https://www.trustedparts.com/en/search/FW-03-03-G-D-085-155"
+			(at 256.54 102.87 0)
 			(show_name yes)
 			(effects
@@
 		)
 		(property "Voltage Rating (V)" "300"
-			(at 256.54 104.14 0)
+			(at 256.54 105.41 0)
 			(show_name yes)
 			(effects
@@
 		(pin "1"
 		)
+		(pin "6"
+		)
+		(pin "5"
+		)
 		(instances

Commit message: Update KiCAD Symbol Generator submodule and add new footprint and symbol libraries
Parts:
- added M1: ~, mechanical_parts:2907525, symbol UNITED_MECHANICAL_DATA_BASE:M_UM108_PROFIL
- added M2: ~, mechanical_parts:2959696, symbol UNITED_MECHANICAL_DATA_BASE:M_UM108_SEFE_L
- added M3: ~, mechanical_parts:2959683, symbol UNITED_MECHANICAL_DATA_BASE:M_UM108_SEFE_R
Changed lines of the file:
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@@
+	)
+	(symbol
+		(lib_id "UNITED_MECHANICAL_DATA_BASE:M_UM108_SEFE_L")
+		(at 345.44 190.5 0)
+		(unit 1)
+		(exclude_from_sim no)
+		(in_bom yes)
+		(on_board yes)
+		(dnp no)
+		(fields_autoplaced yes)
+		(property "Reference" "M2"
+			(at 350.52 189.8649 0)
+			(effects
+				(font
+					(size 1.27 1.27)
+				)
+				(justify left)
+			)
+		)
+		(property "Value" "~"
+			(at 350.52 191.77 0)
+			(effects
+				(font
+					(size 1.27 1.27)
+				)
+				(justify left)
+			)
+		)
+		(property "Footprint" "mechanical_parts:2959696"
+			(at 345.44 190.5 0)
+			(effects
+				(font
+					(size 1.27 1.27)
+				)
+				(hide yes)
+			)
+		)
+		(property "Datasheet" ""
+			(at 345.44 190.5 0)
+			(effects
+				(font
+					(size 1.27 1.27)
+				)
+				(hide yes)
+			)
+		)
+		(property "Description" ""
+			(at 345.44 190.5 0)
+			(effects
+				(font
+					(size 1.27 1.27)
+				)
+				(hide yes)
+			)
+		)
+		(instances
+			(project ""
+				(path "/b764ffe3-5231-4422-b46d-b0de4c44c7b4"
+					(reference "M2")
+					(unit 1)
+				)
+			)
+		)
 	)
 	(symbol
@@
 					(unit 1)
 				)
+			)
+		)
+	)
+	(symbol
+		(lib_id "UNITED_MECHANICAL_DATA_BASE:M_UM108_SEFE_R")
+		(at 392.43 190.5 0)
+		(unit 1)
+		(exclude_from_sim no)
+		(in_bom yes)
+		(on_board yes)
+		(dnp no)
+		(fields_autoplaced yes)
+		(property "Reference" "M3"
+			(at 397.51 189.8649 0)
+			(effects
+				(font
+					(size 1.27 1.27)
+				)
+				(justify left)
+			)
+		)
+		(property "Value" "~"
+			(at 397.51 191.77 0)
+			(effects
+				(font
+					(size 1.27 1.27)
+				)
+				(justify left)
+			)
+		)
+		(property "Footprint" "mechanical_parts:2959683"
+			(at 392.43 190.5 0)
+			(effects
+				(font
+					(size 1.27 1.27)
+				)
+				(hide yes)
+			)
+		)
+		(property "Datasheet" ""
+			(at 392.43 190.5 0)
+			(effects
+				(font
+					(size 1.27 1.27)
+				)
+				(hide yes)
+			)
+		)
+		(property "Description" ""
+			(at 392.43 190.5 0)
+			(effects
+				(font
+					(size 1.27 1.27)
+				)
+				(hide yes)
+			)
+		)
+		(instances
+			(project ""
+				(path "/b764ffe3-5231-4422-b46d-b0de4c44c7b4"
+					(reference "M3")
+					(unit 1)
+				)
+			)
+		)
+	)
+	(symbol
+		(lib_id "UNITED_MECHANICAL_DATA_BASE:M_UM108_PROFIL")
+		(at 368.3 190.5 0)
+		(unit 1)
+		(exclude_from_sim no)
+		(in_bom yes)
+		(on_board yes)
+		(dnp no)
+		(fields_autoplaced yes)
+		(property "Reference" "M1"
+			(at 382.27 189.8649 0)
+			(effects
+				(font
+					(size 1.27 1.27)
+				)
+				(justify left)
+			)
+		)
+		(property "Value" "~"
+			(at 382.27 191.77 0)
+			(effects
+				(font
+					(size 1.27 1.27)
+				)
+				(justify left)
+			)
+		)
+		(property "Footprint" "mechanical_parts:2907525"
+			(at 368.3 190.5 0)
+			(effects
+				(font
+					(size 1.27 1.27)
+				)
+				(hide yes)
+			)
+		)
+		(property "Datasheet" ""
+			(at 368.3 190.5 0)
+			(effects
+				(font
+					(size 1.27 1.27)
+				)
+				(hide yes)
+			)
+		)
+		(property "Description" ""
+			(at 368.3 190.5 0)
+			(effects
+				(font
+					(size 1.27 1.27)
+				)
+				(hide yes)
+			)
+		)
+		(instances
+			(project ""
+				(path "/b764ffe3-5231-4422-b46d-b0de4c44c7b4"
+					(reference "M1")
+					(unit 1)
+				)

Commit message: Backup
Parts:
- removed J23: TBP02R2-381-08BE, connector_footprints:TBP02R2-381-08BE, symbol UNITED_CONNECTORS_DATA_BASE:J_TBP02R2-381-08BE
Changed lines of the file:
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@@
-	)
-	(symbol
-		(lib_id "UNITED_CONNECTORS_DATA_BASE:J_TBP02R2-381-08BE")
-		(at 177.8 180.34 0)
-		(unit 1)
-		(exclude_from_sim no)
-		(in_bom yes)
-		(on_board yes)
-		(dnp no)
-		(fields_autoplaced yes)
-		(property "Reference" "J23"
-			(at 181.61 179.0699 0)
-			(effects
-				(font
-					(size 1.27 1.27)
-				)
-				(justify left)
-			)
-		)
-		(property "Value" "TBP02R2-381-08BE"
-			(at 181.61 181.6099 0)
-			(effects
-				(font
-					(size 1.27 1.27)
-				)
-				(justify left)
-			)
-		)
-		(property "Footprint" "connector_footprints:TBP02R2-381-08BE"
-			(at 182.88 195.58 0)
-			(show_name yes)
-			(effects
-				(font
-					(size 1.27 1.27)
-				)
-				(justify left)
-				(hide yes)
-			)
-		)
-		(property "Datasheet" "https://www.sameskydevices.com/product/resource/tbp02r2-381.pdf"
-			(at 182.88 198.12 0)
-			(show_name yes)
-			(effects
-				(font
-					(size 1.27 1.27)
-				)
-				(justify left)
-				(hide yes)
-			)
-		)
-		(property "Description" "Same Sky TBP02R2-381 series,  8 positions connector,  3.81 mm pitch,  Blue,  Vertical mounting,  8.0 A,  300 V,  Through Hole,  Tin plated"
-			(at 182.88 200.66 0)
-			(show_name yes)
-			(effects
-				(font
-					(size 1.27 1.27)
-				)
-				(justify left)
-				(hide yes)
-			)
-		)
-		(property "Color" "Blue"
-			(at 182.88 203.2 0)
-			(show_name yes)
-			(effects
-				(font
-					(size 1.27 1.27)
-				)
-				(justify left)
-				(hide yes)
-			)
-		)
-		(property "Contact Plating" "Tin"
-			(at 182.88 205.74 0)
-			(show_name yes)
-			(effects
-				(font
-					(size 1.27 1.27)
-				)
-				(justify left)
-				(hide yes)
-			)
-		)
-		(property "Current Rating (A)" "8.0"
-			(at 182.88 208.28 0)
-			(show_name yes)
-			(effects
-				(font
-					(size 1.27 1.27)
-				)
-				(justify left)
-				(hide yes)
-			)
-		)
-		(property "MPN" "TBP02R2-381-08BE"
-			(at 182.88 210.82 0)
-			(show_name yes)
-			(effects
-				(font
-					(size 1.27 1.27)
-				)
-				(justify left)
-				(hide yes)
-			)
-		)
-		(property "Manufacturer" "Same Sky"
-			(at 182.88 213.36 0)
-			(show_name yes)
-			(effects
-				(font
-					(size 1.27 1.27)
-				)
-				(justify left)
-				(hide yes)
-			)
-		)
-		(property "Mounting Angle" "Vertical"
-			(at 182.88 215.9 0)
-			(show_name yes)
-			(effects
-				(font
-					(size 1.27 1.27)
-				)
-				(justify left)
-				(hide yes)
-			)
-		)
-		(property "Mounting Style" "Through Hole"
-			(at 182.88 218.44 0)
-			(show_name yes)
-			(effects
-				(font
-					(size 1.27 1.27)
-				)
-				(justify left)
-				(hide yes)
-			)
-		)
-		(property "Number of Rows" "1"
-			(at 182.88 220.98 0)
-			(show_name yes)
-			(effects
-				(font
-					(size 1.27 1.27)
-				)
-				(justify left)
-				(hide yes)
-			)
-		)
-		(property "Pin Count" "8"
-			(at 182.88 223.52 0)
-			(show_name yes)
-			(effects
-				(font
-					(size 1.27 1.27)
-				)
-				(justify left)
-				(hide yes)
-			)
-		)
-		(property "Pitch (mm)" "3.81"
-			(at 182.88 226.06 0)
-			(show_name yes)
-			(effects
-				(font
-					(size 1.27 1.27)
-				)
-				(justify left)
-				(hide yes)
-			)
-		)
-		(property "Series" "TBP02R2-381"
-			(at 182.88 228.6 0)
-			(show_name yes)
-			(effects
-				(font
-					(size 1.27 1.27)
-				)
-				(justify left)
-				(hide yes)
-			)
-		)
-		(property "Symbol Name" "J_TBP02R2-381-08BE"
-			(at 182.88 231.14 0)
-			(show_name yes)
-			(effects
-				(font
-					(size 1.27 1.27)
-				)
-				(justify left)
-				(hide yes)
-			)
-		)
-		(property "Trustedparts Search" "https://www.trustedparts.com/en/search/TBP02R2-381-08BE"
-			(at 182.88 233.68 0)
-			(show_name yes)
-			(effects
-				(font
-					(size 1.27 1.27)
-				)
-				(justify left)
-				(hide yes)
-			)
-		)
-		(property "Voltage Rating (V)" "300"
-			(at 182.88 236.22 0)
-			(show_name yes)
-			(effects
-				(font
-					(size 1.27 1.27)
-				)
-				(justify left)
-				(hide yes)
-			)
-		)
-		(pin "3"
-		)
-		(pin "8"
-		)
-		(pin "5"
-		)
-		(pin "1"
-		)
-		(pin "4"
-		)
-		(pin "7"
-		)
-		(pin "2"
-		)
-		(pin "6"
-		)
-		(instances
-			(project ""
-				(path "/b764ffe3-5231-4422-b46d-b0de4c44c7b4"
-					(reference "J23")
-					(unit 1)
-				)
-			)
-		)
 	)
 	(symbol

Commit message: Update KiCAD Symbol Generator submodule and add new mechanical component symbols
Parts:
- added M12, M13, M4, M5, M6, M7: ~, mechanical_parts:9774020243R, symbol UNITED_MECHANICAL_DATA_BASE:M_9774020243R
