File: modular_software_configurable_io_plc/modular_software_configurable_io_plc.kicad_sch (KiCad schematic)
At the start: 42 parts, among them J1 FW-09-03-G-D-085-155, J15 FW-14-03-G-D-085-155, J16 FW-02-03-G-D-085-155, J17 FW-02-03-G-D-085-155, J18 FW-02-03-G-D-085-155, J19 FW-02-03-G-D-085-155, J2 CLP-102-02-G-D-BE, J20 CLP-102-02-G-D-BE, J21 CLP-102-02-G-D-BE, J22 FW-02-03-G-D-085-155, J23 CLP-102-02-G-D-BE, J24 FW-02-03-G-D-085-155, J25 FW-02-03-G-D-085-155, J26 FW-02-03-G-D-085-155, J27 FW-02-03-G-D-085-155, J28 FW-02-03-G-D-085-155, J29 FW-02-03-G-D-085-155, J3 CLP-102-02-G-D-BE, J30 CLP-102-02-G-D-BE, J31 CLP-102-02-G-D-BE, J33 CLP-102-02-G-D-BE, J34 CLP-102-02-G-D-BE, J35 CLP-102-02-G-D-BE, J4 CLP-102-02-G-D-BE, J5 CLP-102-02-G-D-BE, J6 CLP-102-02-G-D-BE, J7 CLP-102-02-G-D-BE, J8 CLP-114-02-G-D-BE, J9 FW-09-03-G-D-085-155

Commit message: development backup
Parts:
- added J36: CLP-103-02-G-D-BE, connector_footprints:CLP-103-02-G-D-BE, symbol UNITED_CONNECTORS_DATA_BASE:J_CLP-103-02-G-D-BE
Changed lines of the file:
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@@
+	)
+	(symbol
+		(lib_id "UNITED_CONNECTORS_DATA_BASE:J_CLP-103-02-G-D-BE")
+		(at 321.31 97.79 0)
+		(mirror y)
+		(unit 1)
+		(exclude_from_sim no)
+		(in_bom yes)
+		(on_board yes)
+		(dnp no)
+		(fields_autoplaced yes)
+		(property "Reference" "J36"
+			(at 321.31 87.63 0)
+			(effects
+				(font
+					(size 1.27 1.27)
+				)
+			)
+		)
+		(property "Value" "CLP-103-02-G-D-BE"
+			(at 321.31 90.17 0)
+			(effects
+				(font
+					(size 1.27 1.27)
+				)
+			)
+		)
+		(property "Footprint" "connector_footprints:CLP-103-02-G-D-BE"
+			(at 316.23 106.68 0)
+			(show_name yes)
+			(effects
+				(font
+					(size 1.27 1.27)
+				)
+				(justify left)
+				(hide yes)
+			)
+		)
+		(property "Datasheet" "https://suddendocs.samtec.com/catalog_english/clp_sm.pdf?_gl=1*1y4jlr9*_gcl_au*MTM0MTYyNTQ5MS4xNzM2MDk5MTUz*_ga*MTYxNDYyMTQ0Mi4xNzM2MDk5MTUz*_ga_3KFNZC07WW*MTczNjY4MDQ4OS4xNS4xLjE3MzY2ODEzNzcuNjAuMC4w"
+			(at 316.23 109.22 0)
+			(show_name yes)
+			(effects
+				(font
+					(size 1.27 1.27)
+				)
+				(justify left)
+				(hide yes)
+			)
+		)
+		(property "Description" "Samtec CLP-1xx-02-G-D-BE series,  3 positions connector,  1.27 mm pitch,  Black,  Vertical mounting,  5.2 A,  300 V,  Surface Mount,  Tin plated"
+			(at 316.23 111.76 0)
+			(show_name yes)
+			(effects
+				(font
+					(size 1.27 1.27)
+				)
+				(justify left)
+				(hide yes)
+			)
+		)
+		(property "Color" "Black"
+			(at 316.23 114.3 0)
+			(show_name yes)
+			(effects
+				(font
+					(size 1.27 1.27)
+				)
+				(justify left)
+				(hide yes)
+			)
+		)
+		(property "Contact Plating" "Tin"
+			(at 316.23 116.84 0)
+			(show_name yes)
+			(effects
+				(font
+					(size 1.27 1.27)
+				)
+				(justify left)
+				(hide yes)
+			)
+		)
+		(property "Current Rating (A)" "5.2"
+			(at 316.23 119.38 0)
+			(show_name yes)
+			(effects
+				(font
+					(size 1.27 1.27)
+				)
+				(justify left)
+				(hide yes)
+			)
+		)
+		(property "MPN" "CLP-103-02-G-D-BE"
+			(at 316.23 121.92 0)
+			(show_name yes)
+			(effects
+				(font
+					(size 1.27 1.27)
+				)
+				(justify left)
+				(hide yes)
+			)
+		)
+		(property "Manufacturer" "Samtec"
+			(at 316.23 124.46 0)
+			(show_name yes)
+			(effects
+				(font
+					(size 1.27 1.27)
+				)
+				(justify left)
+				(hide yes)
+			)
+		)
+		(property "Mounting Angle" "Vertical"
+			(at 316.23 127 0)
+			(show_name yes)
+			(effects
+				(font
+					(size 1.27 1.27)
+				)
+				(justify left)
+				(hide yes)
+			)
+		)
+		(property "Mounting Style" "Surface Mount"
+			(at 316.23 129.54 0)
+			(show_name yes)
+			(effects
+				(font
+					(size 1.27 1.27)
+				)
+				(justify left)
+				(hide yes)
+			)
+		)
+		(property "Number of Rows" "2"
+			(at 316.23 132.08 0)
+			(show_name yes)
+			(effects
+				(font
+					(size 1.27 1.27)
+				)
+				(justify left)
+				(hide yes)
+			)
+		)
+		(property "Pin Count" "3"
+			(at 316.23 134.62 0)
+			(show_name yes)
+			(effects
+				(font
+					(size 1.27 1.27)
+				)
+				(justify left)
+				(hide yes)
+			)
+		)
+		(property "Pitch (mm)" "1.27"
+			(at 316.23 137.16 0)
+			(show_name yes)
+			(effects
+				(font
+					(size 1.27 1.27)
+				)
+				(justify left)
+				(hide yes)
+			)
+		)
+		(property "Series" "CLP-1xx-02-G-D-BE"
+			(at 316.23 139.7 0)
+			(show_name yes)
+			(effects
+				(font
+					(size 1.27 1.27)
+				)
+				(justify left)
+				(hide yes)
+			)
+		)
+		(property "Symbol Name" "J_CLP-103-02-G-D-BE"
+			(at 316.23 142.24 0)
+			(show_name yes)
+			(effects
+				(font
+					(size 1.27 1.27)
+				)
+				(justify left)
+				(hide yes)
+			)
+		)
+		(property "Trustedparts Search" "https://www.trustedparts.com/en/search/CLP-103-02-G-D-BE"
+			(at 316.23 144.78 0)
+			(show_name yes)
+			(effects
+				(font
+					(size 1.27 1.27)
+				)
+				(justify left)
+				(hide yes)
+			)
+		)
+		(property "Voltage Rating (V)" "300"
+			(at 316.23 147.32 0)
+			(show_name yes)
+			(effects
+				(font
+					(size 1.27 1.27)
+				)
+				(justify left)
+				(hide yes)
+			)
+		)
+		(pin "1"
+		)
+		(pin "4"
+		)
+		(pin "2"
+		)
+		(pin "3"
+		)
+		(pin "5"
+		)
+		(pin "6"
+		)
+		(instances
+			(project "modular_software_configurable_io_plc"
+				(path "/b764ffe3-5231-4422-b46d-b0de4c44c7b4"
+					(reference "J36")
+					(unit 1)
+				)
+			)
+		)
 	)
 	(symbol

Commit message: development backup
Parts:
- removed M12, M13, M6, M7: ~, mechanical_parts:9774020243R, symbol UNITED_MECHANICAL_DATA_BASE:M_9774020243R

Commit message: development backup
Parts:
- added J10: TBP04R2-500-02BE, connector_footprints:TBP04R2-500-02BE, symbol UNITED_CONNECTORS_DATA_BASE:J_TBP04R2-500-02BE
- added J11: TBP02R2-381-03BE, connector_footprints:TBP02R2-381-03BE, symbol UNITED_CONNECTORS_DATA_BASE:J_TBP02R2-381-03BE
- added J12, J13, J14, J37: TBP02R2-381-02BE, connector_footprints:TBP02R2-381-02BE, symbol UNITED_CONNECTORS_DATA_BASE:J_TBP02R2-381-02BE

Commit message: development backup
Parts:
- removed J24: FW-02-03-G-D-085-155, connector_footprints:FW-02-03-G-D-085-155, symbol UNITED_CONNECTORS_DATA_BASE:J_FW-02-03-G-D-085-155
- added S1: 8SS1012-Z, switches_footprints:8SS1012-Z, symbol UNITED_SWITCHES_DATA_BASE:S_8SS1012-Z
- J29: value FW-02-03-G-D-085-155 -> FW-05-03-G-D-085-155; footprint connector_footprints:FW-02-03-G-D-085-155 -> connector_footprints:FW-05-03-G-D-085-155; symbol UNITED_CONNECTORS_DATA_BASE:J_FW-02-03-G-D-085-155 -> UNITED_CONNECTORS_DATA_BASE:J_FW-05-03-G-D-085-155; MPN FW-02-03-G-D-085-155 -> FW-05-03-G-D-085-155; Pin Count 2 -> 5; Symbol Name J_FW-02-03-G-D-085-155 -> J_FW-05-03-G-D-085-155; Trustedparts Search https://www.trustedparts.com/en/search/FW-02-03-G-D-085-155 -> https://www.trustedparts.com/en/search/FW-05-03-G-D-085-155

Commit message: development backup
Parts:
- removed J1, J9: FW-09-03-G-D-085-155, connector_footprints:FW-09-03-G-D-085-155, symbol UNITED_CONNECTORS_DATA_BASE:J_FW-09-03-G-D-085-155
- removed J15: FW-14-03-G-D-085-155, connector_footprints:FW-14-03-G-D-085-155, symbol UNITED_CONNECTORS_DATA_BASE:J_FW-14-03-G-D-085-155
- removed J16, J17, J18, J19, J22, J25, J26, J27, J28: FW-02-03-G-D-085-155, connector_footprints:FW-02-03-G-D-085-155, symbol UNITED_CONNECTORS_DATA_BASE:J_FW-02-03-G-D-085-155
- removed J2, J20, J21, J23, J3, J30, J31, J33, J34, J35, J4, J5, J6, J7: CLP-102-02-G-D-BE, connector_footprints:CLP-102-02-G-D-BE, symbol UNITED_CONNECTORS_DATA_BASE:J_CLP-102-02-G-D-BE
- removed J29: FW-05-03-G-D-085-155, connector_footprints:FW-05-03-G-D-085-155, symbol UNITED_CONNECTORS_DATA_BASE:J_FW-05-03-G-D-085-155
- removed J36: CLP-103-02-G-D-BE, connector_footprints:CLP-103-02-G-D-BE, symbol UNITED_CONNECTORS_DATA_BASE:J_CLP-103-02-G-D-BE
- removed J8: CLP-114-02-G-D-BE, connector_footprints:CLP-114-02-G-D-BE, symbol UNITED_CONNECTORS_DATA_BASE:J_CLP-114-02-G-D-BE
- removed MOD1: ~, modules_footprints:minimal_ad74413r, symbol UNITED_MODULES_DATA_BASE:MINIMAL_AD74413R
- removed MOD2: ~, modules_footprints:minimal_max14906, symbol UNITED_MODULES_DATA_BASE:MINIMAL_MAX14906
- removed MOD4: ~, modules_footprints:minimal_adin1110, symbol UNITED_MODULES_DATA_BASE:MINIMAL_ADIN1110
- removed MOD5: ~, modules_footprints:minimal_ltc9111, symbol UNITED_MODULES_DATA_BASE:MINIMAL_LTC9111
- removed MOD7: ~, modules_footprints:minimal_max17761, symbol UNITED_MODULES_DATA_BASE:MINIMAL_MAX17761
- removed MOD8: ~, modules_footprints:minimal_lt8304, symbol UNITED_MODULES_DATA_BASE:MINIMAL_LT8304
Other:
- added sheet Minimal_AD74413R (Minimal_AD74413R.kicad_sch)
- added sheet Minimal_ADIN1110 (Minimal_ADIN1110.kicad_sch)
- added sheet Minimal_LT8304 (Minimal_LT8304.kicad_sch)
- added sheet Minimal_LTC9111 (Minimal_LTC9111.kicad_sch)
- added sheet Minimal_MAX14906 (Minimal_MAX14906.kicad_sch)
- moved on the sheet: J10

Commit message: development backup
Parts:
- added FID1, FID2, FID3: Fiducial, no_components_footprints:Fiducial_0.5mm_Mask1mm, symbol UNITED_NO_COMPONENTS_DATA_BASE:Fiducial
Changed lines of the file:
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@@
 	(paper "A3")
+	(symbol
+		(lib_id "UNITED_NO_COMPONENTS_DATA_BASE:Fiducial")
+		(at 355.6 215.9 0)
+		(unit 1)
+		(exclude_from_sim no)
+		(in_bom yes)
+		(on_board yes)
+		(dnp no)
+		(fields_autoplaced yes)
+		(property "Reference" "FID1"
+			(at 358.14 214.6299 0)
+			(effects
+				(font
+					(size 1.27 1.27)
+				)
+				(justify left)
+			)
+		)
+		(property "Value" "Fiducial"
+			(at 358.14 217.1699 0)
+			(effects
+				(font
+					(size 1.27 1.27)
+				)
+				(justify left)
+			)
+		)
+		(property "Footprint" "no_components_footprints:Fiducial_0.5mm_Mask1mm"
+			(at 355.6 223.52 0)
+			(effects
+				(font
+					(size 1.27 1.27)
+				)
+				(justify left)
+				(hide yes)
+			)
+		)
+		(property "Datasheet" "~"
+			(at 355.6 218.44 0)
+			(effects
+				(font
+					(size 1.27 1.27)
+				)
+				(justify left)
+				(hide yes)
+			)
+		)
+		(property "Description" "Fiducial Marker"
+			(at 355.6 220.98 0)
+			(effects
+				(font
+					(size 1.27 1.27)
+				)
+				(justify left)
+				(hide yes)
+			)
+		)
+		(instances
+			(project ""
+				(path "/b764ffe3-5231-4422-b46d-b0de4c44c7b4"
+					(reference "FID1")
+					(unit 1)
+				)
+			)
+		)
+	)
 	(symbol
 		(lib_id "UNITED_CONNECTORS_DATA_BASE:J_TBP02R2-381-02BE")
@@
 	)
 	(symbol
+		(lib_id "UNITED_NO_COMPONENTS_DATA_BASE:Fiducial")
+		(at 368.3 215.9 0)
+		(unit 1)
+		(exclude_from_sim no)
+		(in_bom yes)
+		(on_board yes)
+		(dnp no)
+		(fields_autoplaced yes)
+		(property "Reference" "FID2"
+			(at 370.84 214.6299 0)
+			(effects
+				(font
+					(size 1.27 1.27)
+				)
+				(justify left)
+			)
+		)
+		(property "Value" "Fiducial"
+			(at 370.84 217.1699 0)
+			(effects
+				(font
+					(size 1.27 1.27)
+				)
+				(justify left)
+			)
+		)
+		(property "Footprint" "no_components_footprints:Fiducial_0.5mm_Mask1mm"
+			(at 368.3 223.52 0)
+			(effects
+				(font
+					(size 1.27 1.27)
+				)
+				(justify left)
+				(hide yes)
+			)
+		)
+		(property "Datasheet" "~"
+			(at 368.3 218.44 0)
+			(effects
+				(font
+					(size 1.27 1.27)
+				)
+				(justify left)
+				(hide yes)
+			)
+		)
+		(property "Description" "Fiducial Marker"
+			(at 368.3 220.98 0)
+			(effects
+				(font
+					(size 1.27 1.27)
+				)
+				(justify left)
+				(hide yes)
+			)
+		)
+		(instances
+			(project "modular_software_configurable_io_plc"
+				(path "/b764ffe3-5231-4422-b46d-b0de4c44c7b4"
+					(reference "FID2")
+					(unit 1)
+				)
+			)
+		)
+	)
+	(symbol
 		(lib_id "UNITED_MECHANICAL_DATA_BASE:M_UM108_SEFE_R")
 		(at 392.43 190.5 0)
@@
 					(unit 1)
 				)
+			)
+		)
+	)
+	(symbol
+		(lib_id "UNITED_NO_COMPONENTS_DATA_BASE:Fiducial")
+		(at 381 215.9 0)
+		(unit 1)
+		(exclude_from_sim no)
+		(in_bom yes)
+		(on_board yes)
+		(dnp no)
+		(fields_autoplaced yes)
+		(property "Reference" "FID3"
+			(at 383.54 214.6299 0)
+			(effects
+				(font
+					(size 1.27 1.27)
+				)
+				(justify left)
+			)
+		)
+		(property "Value" "Fiducial"
+			(at 383.54 217.1699 0)
+			(effects
+				(font
+					(size 1.27 1.27)
+				)
+				(justify left)
+			)
+		)
+		(property "Footprint" "no_components_footprints:Fiducial_0.5mm_Mask1mm"
+			(at 381 223.52 0)
+			(effects
+				(font
+					(size 1.27 1.27)
+				)
+				(justify left)
+				(hide yes)
+			)
+		)
+		(property "Datasheet" "~"
+			(at 381 218.44 0)
+			(effects
+				(font
+					(size 1.27 1.27)
+				)
+				(justify left)
+				(hide yes)
+			)
+		)
+		(property "Description" "Fiducial Marker"
+			(at 381 220.98 0)
+			(effects
+				(font
+					(size 1.27 1.27)
+				)
+				(justify left)
+				(hide yes)
+			)
+		)
+		(instances
+			(project "modular_software_configurable_io_plc"
+				(path "/b764ffe3-5231-4422-b46d-b0de4c44c7b4"
+					(reference "FID3")
+					(unit 1)
+				)

Commit message: Backup
Parts:
- S1: footprint switches_footprints:8SS1012-Z -> slide_switches_footprints:8SS1012-Z; symbol UNITED_SWITCHES_DATA_BASE:S_8SS1012-Z -> SLIDE_SWITCHES_8SS1012-Z_DATA_BASE:S_8SS1012-Z; Manufacturer (none) -> Nidec Components Corporation; Mounting Angle (none) -> Vertical; Mounting Style (none) -> Through Hole; Number of Rows (none) -> 1; Pin Count (none) -> 3; Series (none) -> 8SS1012-Z; Symbol Name (none) -> S_8SS1012-Z; Trustedparts Search (none) -> https://www.trustedparts.com/en/search/8SS1012-Z
Changed lines of the file:
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@@
 	)
 	(symbol
-		(lib_id "UNITED_SWITCHES_DATA_BASE:S_8SS1012-Z")
+		(lib_id "SLIDE_SWITCHES_8SS1012-Z_DATA_BASE:S_8SS1012-Z")
 		(at 233.68 231.14 0)
 		(unit 1)
@@
 			)
 		)
-		(property "Footprint" "switches_footprints:8SS1012-Z"
-			(at 233.68 241.3 0)
+		(property "Footprint" "slide_switches_footprints:8SS1012-Z"
+			(at 233.68 238.76 0)
+			(show_name yes)
 			(effects
 				(font
@@
 		)
 		(property "Datasheet" "https://www.nidec-components.com/e/catalog/switch/8ss.pdf"
-			(at 233.68 236.22 0)
+			(at 233.68 241.3 0)
+			(show_name yes)
 			(effects
 				(font
@@
 			)
 		)
-		(property "Description" "SWITCH SLIDE SPDT 6A 125V"
-			(at 233.68 238.76 0)
+		(property "Description" "Nidec Components Corporation Vertical mounting,  Through Hole,"
+			(at 233.68 243.84 0)
+			(show_name yes)
 			(effects
 				(font
@@
 		)
 		(property "MPN" "8SS1012-Z"
-			(at 233.68 243.84 0)
+			(at 233.68 246.38 0)
+			(show_name yes)
 			(effects
 				(font
+					(size 1.27 1.27)
+				)
+				(justify left)
+				(hide yes)
+			)
+		)
+		(property "Manufacturer" "Nidec Components Corporation"
+			(at 233.68 248.92 0)
+			(effects
+				(font
+					(size 1.27 1.27)
+				)
+				(justify left)
+				(hide yes)
+			)
+		)
+		(property "Mounting Angle" "Vertical"
+			(at 233.68 251.46 0)
+			(effects
+				(font
+					(size 1.27 1.27)
+				)
+				(justify left)
+				(hide yes)
+			)
+		)
+		(property "Mounting Style" "Through Hole"
+			(at 233.68 254 0)
+			(effects
+				(font
+					(size 1.27 1.27)
+				)
+				(justify left)
+				(hide yes)
+			)
+		)
+		(property "Number of Rows" "1"
+			(at 233.68 256.54 0)
+			(effects
+				(font
+					(size 1.27 1.27)
+				)
+				(justify left)
+				(hide yes)
+			)
+		)
+		(property "Pin Count" "3"
+			(at 233.68 259.08 0)
+			(effects
+				(font
+					(size 1.27 1.27)
+				)
+				(justify left)
+				(hide yes)
+			)
+		)
+		(property "Series" "8SS1012-Z"
+			(at 233.68 261.62 0)
+			(effects
+				(font
+					(size 1.27 1.27)
+				)
+				(justify left)
+				(hide yes)
+			)
+		)
+		(property "Symbol Name" "S_8SS1012-Z"
+			(at 233.68 264.16 0)
+			(effects
+				(font
+					(size 1.27 1.27)
+				)
+				(justify left)
+				(hide yes)
+			)
+		)
+		(property "Trustedparts Search" "https://www.trustedparts.com/en/search/8SS1012-Z"
+			(at 233.68 266.7 0)
+			(effects
+				(font

Commit message: Backup
Parts:
- renumbered J10 to J2, J14 to J23, J12 to J24, J11 to J3, J37 to J30, J13 to J31, M2 to M1, M1 to M2
Changed lines of the file:
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@@
 		(dnp no)
 		(fields_autoplaced yes)
-		(property "Reference" "J37"
+		(property "Reference" "J30"
 			(at 243.84 184.1499 0)
 			(effects
@@
 			(project "modular_software_configurable_io_plc"
 				(path "/b764ffe3-5231-4422-b46d-b0de4c44c7b4"
-					(reference "J37")
+					(reference "J30")
 					(unit 1)
 				)
@@
 		(on_board yes)
 		(dnp no)
-		(property "Reference" "J10"
+		(property "Reference" "J2"
 			(at 57.15 124.4599 0)
 			(effects
@@
 			(project "modular_software_configurable_io_plc"
 				(path "/b764ffe3-5231-4422-b46d-b0de4c44c7b4"
-					(reference "J10")
+					(reference "J2")
 					(unit 1)
 				)
@@
 		(dnp no)
 		(fields_autoplaced yes)
-		(property "Reference" "M2"
+		(property "Reference" "M1"
 			(at 350.52 189.8649 0)
 			(effects
@@
 			(project ""
 				(path "/b764ffe3-5231-4422-b46d-b0de4c44c7b4"
-					(reference "M2")
+					(reference "M1")
 					(unit 1)
 				)
@@
 		(dnp no)
 		(fields_autoplaced yes)
-		(property "Reference" "J13"
+		(property "Reference" "J31"
 			(at 208.28 195.5799 0)
 			(effects
@@
 			(project "modular_software_configurable_io_plc"
 				(path "/b764ffe3-5231-4422-b46d-b0de4c44c7b4"
-					(reference "J13")
+					(reference "J31")
 					(unit 1)
 				)
@@
 		(dnp no)
 		(fields_autoplaced yes)
-		(property "Reference" "J11"
+		(property "Reference" "J3"
 			(at 254 153.6699 0)
 			(effects
@@
 			(project ""
 				(path "/b764ffe3-5231-4422-b46d-b0de4c44c7b4"
-					(reference "J11")
+					(reference "J3")
 					(unit 1)
 				)
@@
 		(dnp no)
 		(fields_autoplaced yes)
-		(property "Reference" "M1"
+		(property "Reference" "M2"
 			(at 382.27 189.8649 0)
 			(effects
@@
 			(project ""
 				(path "/b764ffe3-5231-4422-b46d-b0de4c44c7b4"
-					(reference "M1")
+					(reference "M2")
 					(unit 1)
 				)
@@
 		(dnp no)
 		(fields_autoplaced yes)
-		(property "Reference" "J12"
+		(property "Reference" "J24"
 			(at 205.74 184.1499 0)
 			(effects
@@
 			(project ""
 				(path "/b764ffe3-5231-4422-b46d-b0de4c44c7b4"
-					(reference "J12")
+					(reference "J24")
 					(unit 1)
 				)
@@
 		(dnp no)
 		(fields_autoplaced yes)
-		(property "Reference" "J14"
+		(property "Reference" "J23"
 			(at 243.84 195.5799 0)
 			(effects
@@
 			(project "modular_software_configurable_io_plc"
 				(path "/b764ffe3-5231-4422-b46d-b0de4c44c7b4"
-					(reference "J14")
+					(reference "J23")
 					(unit 1)
 				)
