File: modular_software_configurable_io_plc/modular_software_configurable_io_plc.kicad_pcb (KiCad board)
At the start: 4 copper layers, 105 x 107 mm, 43 parts, among them J1 FW-09-03-G-D-085-155, J15 FW-14-03-G-D-085-155, J16 FW-02-03-G-D-085-155, J17 FW-02-03-G-D-085-155, J18 FW-02-03-G-D-085-155, J19 FW-02-03-G-D-085-155, J2 CLP-102-02-G-D-BE, J20 CLP-102-02-G-D-BE, J21 CLP-103-02-G-D-BE, J22 FW-02-03-G-D-085-155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

Commit message: development backup
Parts:
- added J35: CLP-102-02-G-D-BE, connector_footprints:CLP-102-02-G-D-BE, F.Cu at (118.7, 99.5)
- J21: value CLP-103-02-G-D-BE -> CLP-102-02-G-D-BE; footprint connector_footprints:CLP-103-02-G-D-BE -> connector_footprints:CLP-102-02-G-D-BE
- J33: value FW-02-03-G-D-085-155 -> CLP-102-02-G-D-BE; footprint connector_footprints:FW-02-03-G-D-085-155 -> connector_footprints:CLP-102-02-G-D-BE
- moved J30 6.28 mm to (163.8, 49.0)
- moved J23 6.28 mm to (190.2, 49.0)
- moved MOD7 6.28 mm to (177.0, 48.4)
- moved J21 5.95 mm to (108.5, 99.5)
- moved MOD5 2.65 mm to (113.6, 72.1)
- moved J31 1.70 mm to (153.9, 46.5)
- moved J34 1.70 mm to (145.6, 97.9), turned to -90 degrees
- moved MOD8 1.70 mm to (145.6, 71.1)
- moved J15 1.03 mm to (113.6, 64.4)
- moved J17 1.03 mm to (127.6, 84.1)
- moved J18 1.03 mm to (127.6, 75.8)
- moved J19 1.03 mm to (104.9, 101.6)
- moved J22 1.03 mm to (122.4, 101.6)
- moved MOD4 1.03 mm to (116.8, 93.6)
- moved J16 1.03 mm to (127.6, 92.3)
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
Commit message: development backup
Parts:
- moved J20 110.8 mm to (191.1, 123.9), turned to 90 degrees
- moved J19 101.1 mm to (199.8, 66.9), turned to 180 degrees
- moved J21 92.8 mm to (196.2, 69.0), turned to 0 degrees
- moved J15 87.1 mm to (191.1, 104.1), turned to 180 degrees
- moved MOD5 81.2 mm to (191.1, 96.4), turned to 90 degrees
- moved J35 73.9 mm to (186.0, 69.0), turned to 180 degrees
- moved MOD4 73.7 mm to (188.0, 74.9), turned to 90 degrees
- moved J22 69.3 mm to (182.3, 66.9), turned to 0 degrees
- moved J18 52.3 mm to (177.1, 92.7), turned to 0 degrees
- moved J16 52.1 mm to (177.1, 76.2), turned to 0 degrees
- moved J17 49.5 mm to (177.1, 84.4), turned to 0 degrees
- moved J32 28.1 mm to (170.0, 69.8)
- moved MOD9 28.1 mm to (151.3, 69.8)
- moved J23 25.5 mm to (164.7, 48.9)
- moved J30 25.5 mm to (138.3, 48.9)
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
Commit message: development backup
Parts:
- moved J33 15.1 mm to (147.4, 129.5), turned to 90 degrees
- moved J34 14.9 mm to (105.4, 98.4)
- moved MOD8 6.22 mm to (114.3, 72.4)
- moved J31 6.22 mm to (122.6, 47.7)
- moved J2 2.54 mm to (112.9, 136.7), turned to 90 degrees
- moved J3 2.54 mm to (168.7, 136.7), turned to -90 degrees
- moved J4 2.54 mm to (168.7, 106.3)
- moved J5 2.54 mm to (168.7, 116.4)
- moved J6 2.54 mm to (168.7, 126.6)
- moved J7 2.54 mm to (112.9, 126.6)
- moved J8 2.54 mm to (114.8, 105.0)
- moved MOD1 2.54 mm to (140.8, 119.9)
- moved M13 0.32 mm to (174.0, 133.1)
- moved M12 0.32 mm to (174.0, 111.5)
- moved M6 0.32 mm to (107.6, 111.5)
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
Commit message: development backup
Parts:
- added J36: CLP-103-02-G-D-BE, connector_footprints:CLP-103-02-G-D-BE, F.Cu at (191.1, 46.5)
- moved J22 11.4 mm to (187.9, 57.0), turned to 180 degrees
- moved J19 11.4 mm to (194.3, 57.0)
- moved MOD5 10.9 mm to (191.1, 85.5)
- moved J17 7.24 mm to (177.1, 77.2)
- moved J18 7.24 mm to (177.1, 85.5)
- moved J16 7.24 mm to (177.1, 69.0)
- moved J35 4.31 mm to (183.8, 72.7)
- moved J21 4.31 mm to (198.4, 72.7)
- moved J20 2.55 mm to (191.1, 126.4)
- moved J15 2.54 mm to (191.1, 106.7)
- moved MOD4 2.54 mm to (188.0, 77.5)

Commit message: development backup
Parts:
- removed M12, M13, M6, M7: ~, mechanical_parts:9774020243R
- moved J23 31.0 mm to (133.7, 50.5), turned to 90 degrees
- moved J32 30.4 mm to (152.3, 45.2), turned to 0 degrees
- moved J30 28.4 mm to (133.7, 76.9), turned to -90 degrees
- moved MOD7 24.0 mm to (133.1, 63.7), turned to -90 degrees
- moved J18 23.2 mm to (177.1, 108.7)
- moved J19 23.2 mm to (194.3, 80.2)
- moved J22 23.2 mm to (187.9, 80.2)
- moved J16 23.2 mm to (177.1, 92.2)
- moved J17 23.2 mm to (177.1, 100.4)
- moved MOD4 23.2 mm to (188.0, 100.7)
- moved J20 17.4 mm to (191.1, 143.8)
- moved J21 17.4 mm to (198.4, 90.1)
- moved J35 17.4 mm to (183.8, 90.1)
- moved J36 17.4 mm to (191.1, 63.9)
- moved MOD5 17.4 mm to (191.1, 102.9)
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
Commit message: development backup
Parts:
- moved J19 0.64 mm to (193.6, 80.2)
- moved J22 0.64 mm to (187.3, 80.2)
- moved J15 0.63 mm to (190.4, 120.1)
- moved J16 0.63 mm to (177.7, 92.2)
- moved J17 0.63 mm to (177.7, 100.4)
- moved J18 0.63 mm to (177.7, 108.7)

Commit message: development backup
Parts:
- added J10: TBP04R2-500-02BE, connector_footprints:TBP04R2-500-02BE, F.Cu at (121.3, 54.5)
- added J11: TBP02R2-381-03BE, connector_footprints:TBP02R2-381-03BE, F.Cu at (191.3, 55.5)
- added J12: TBP02R2-381-02BE, connector_footprints:TBP02R2-381-02BE, F.Cu at (174.1, 118.6)
- added J13: TBP02R2-381-02BE, connector_footprints:TBP02R2-381-02BE, F.Cu at (174.1, 128.3)
- added J14: TBP02R2-381-02BE, connector_footprints:TBP02R2-381-02BE, F.Cu at (107.3, 118.6)
- added J37: TBP02R2-381-02BE, connector_footprints:TBP02R2-381-02BE, F.Cu at (107.3, 128.3)
- moved J30 43.1 mm to (176.1, 69.4), turned to 0 degrees
- moved J32 38.3 mm to (155.4, 83.4), turned to 180 degrees
- moved MOD7 30.5 mm to (162.9, 70.1), turned to 0 degrees
- moved J23 24.8 mm to (149.7, 69.4), turned to 180 degrees
- moved MOD9 3.14 mm to (155.4, 64.7), turned to 0 degrees
- moved J31 1.27 mm to (121.3, 45.5), turned to -90 degrees
- moved J34 1.27 mm to (104.1, 97.5)
- moved MOD8 1.27 mm to (113.0, 71.5)
- moved J16 0.89 mm to (178.6, 92.2)
- moved J17 0.89 mm to (178.6, 100.4)
- moved J18 0.89 mm to (178.6, 108.7)
- moved J19 0.89 mm to (194.5, 80.2)
- moved J22 0.89 mm to (188.2, 80.2)
- moved MOD4 0.89 mm to (188.9, 100.7)
- moved J15 0.89 mm to (191.3, 120.1)
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
Commit message: development backup
Parts:
- moved J2 0.57 mm to (112.8, 129.5)
- moved J3 0.57 mm to (168.6, 129.5)
- moved J6 0.57 mm to (168.6, 120.6)
- moved J7 0.57 mm to (112.8, 120.6)
- moved J4 0.38 mm to (168.6, 101.2)
- moved J5 0.38 mm to (168.6, 111.4)
- moved J8 0.38 mm to (114.7, 106.4)
- moved MOD1 0.38 mm to (140.7, 116.8)
