File: modular_software_configurable_io_plc/Minimal_AD74413R.kicad_sch (KiCad schematic)
At the start: 8 parts, among them J2 CLP-102-02-G-D-BE, J3 CLP-102-02-G-D-BE, J4 CLP-102-02-G-D-BE, J5 CLP-102-02-G-D-BE, J6 CLP-102-02-G-D-BE, J7 CLP-102-02-G-D-BE, J8 CLP-114-02-G-D-BE

Commit message: Backup
Parts:
- renumbered J4 to J15, J8 to J17, J5 to J20, J7 to J25, J6 to J26, J2 to J32, J3 to J33, MOD1 to MOD6
Changed lines of the file:
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@@
 		(dnp no)
 		(fields_autoplaced yes)
-		(property "Reference" "J3"
+		(property "Reference" "J33"
 			(at 173.99 58.42 0)
 			(effects
@@
 			(project "modular_software_configurable_io_plc"
 				(path "/b764ffe3-5231-4422-b46d-b0de4c44c7b4/30006d44-0996-4923-a210-c99e7b61b211"
-					(reference "J3")
+					(reference "J33")
 					(unit 1)
 				)
@@
 		(dnp no)
 		(fields_autoplaced yes)
-		(property "Reference" "J8"
+		(property "Reference" "J17"
 			(at 132.08 132.0799 90)
 			(effects
@@
 			(project "modular_software_configurable_io_plc"
 				(path "/b764ffe3-5231-4422-b46d-b0de4c44c7b4/30006d44-0996-4923-a210-c99e7b61b211"
-					(reference "J8")
+					(reference "J17")
 					(unit 1)
 				)
@@
 		(on_board yes)
 		(dnp no)
-		(property "Reference" "J6"
+		(property "Reference" "J26"
 			(at 123.19 104.14 0)
 			(effects
@@
 			(project "modular_software_configurable_io_plc"
 				(path "/b764ffe3-5231-4422-b46d-b0de4c44c7b4/30006d44-0996-4923-a210-c99e7b61b211"
-					(reference "J6")
+					(reference "J26")
 					(unit 1)
 				)
@@
 		(dnp no)
 		(fields_autoplaced yes)
-		(property "Reference" "J4"
+		(property "Reference" "J15"
 			(at 123.19 81.28 0)
 			(effects
@@
 			(project "modular_software_configurable_io_plc"
 				(path "/b764ffe3-5231-4422-b46d-b0de4c44c7b4/30006d44-0996-4923-a210-c99e7b61b211"
-					(reference "J4")
+					(reference "J15")
 					(unit 1)
 				)
@@
 		(dnp no)
 		(fields_autoplaced yes)
-		(property "Reference" "MOD1"
+		(property "Reference" "MOD6"
 			(at 153.67 81.28 0)
 			(effects
@@
 			(project "modular_software_configurable_io_plc"
 				(path "/b764ffe3-5231-4422-b46d-b0de4c44c7b4/30006d44-0996-4923-a210-c99e7b61b211"
-					(reference "MOD1")
+					(reference "MOD6")
 					(unit 1)
 				)
@@
 		(dnp no)
 		(fields_autoplaced yes)
-		(property "Reference" "J7"
+		(property "Reference" "J25"
 			(at 173.99 104.14 0)
 			(effects
@@
 			(project "modular_software_configurable_io_plc"
 				(path "/b764ffe3-5231-4422-b46d-b0de4c44c7b4/30006d44-0996-4923-a210-c99e7b61b211"
-					(reference "J7")
+					(reference "J25")
 					(unit 1)
 				)
@@
 		(on_board yes)
 		(dnp no)
-		(property "Reference" "J2"
+		(property "Reference" "J32"
 			(at 123.19 58.42 0)
 			(effects
@@
 			(project "modular_software_configurable_io_plc"
 				(path "/b764ffe3-5231-4422-b46d-b0de4c44c7b4/30006d44-0996-4923-a210-c99e7b61b211"
-					(reference "J2")
+					(reference "J32")
 					(unit 1)
 				)
@@
 		(dnp no)
 		(fields_autoplaced yes)
-		(property "Reference" "J5"
+		(property "Reference" "J20"
 			(at 173.99 81.28 0)
 			(effects
@@
 			(project "modular_software_configurable_io_plc"
 				(path "/b764ffe3-5231-4422-b46d-b0de4c44c7b4/30006d44-0996-4923-a210-c99e7b61b211"
-					(reference "J5")
+					(reference "J20")
 					(unit 1)
 				)
