File: modular_software_configurable_io_plc/Minimal_ADIN1110.kicad_sch (KiCad schematic)
At the start: 7 parts, among them J15 FW-14-03-G-D-085-155, J16 FW-02-03-G-D-085-155, J17 FW-02-03-G-D-085-155, J18 FW-02-03-G-D-085-155, J19 FW-02-03-G-D-085-155, J22 FW-02-03-G-D-085-155

Commit message: Backup
Parts:
- renumbered J16 to J13, J17 to J16, J18 to J19, J15 to J27, J22 to J8, J19 to J9
Changed lines of the file:
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@@
 		(dnp no)
 		(fields_autoplaced yes)
-		(property "Reference" "J15"
+		(property "Reference" "J27"
 			(at 120.65 78.74 0)
 			(effects
@@
 			(project "modular_software_configurable_io_plc"
 				(path "/b764ffe3-5231-4422-b46d-b0de4c44c7b4/aa3cb439-8da3-4fca-ad07-fe00873ec95e"
-					(reference "J15")
+					(reference "J27")
 					(unit 1)
 				)
@@
 		(dnp no)
 		(fields_autoplaced yes)
-		(property "Reference" "J17"
+		(property "Reference" "J16"
 			(at 161.29 78.74 0)
 			(effects
@@
 			(project "modular_software_configurable_io_plc"
 				(path "/b764ffe3-5231-4422-b46d-b0de4c44c7b4/aa3cb439-8da3-4fca-ad07-fe00873ec95e"
-					(reference "J17")
+					(reference "J16")
 					(unit 1)
 				)
@@
 		(dnp no)
 		(fields_autoplaced yes)
-		(property "Reference" "J16"
+		(property "Reference" "J13"
 			(at 143.51 81.28 0)
 			(effects
@@
 			(project "modular_software_configurable_io_plc"
 				(path "/b764ffe3-5231-4422-b46d-b0de4c44c7b4/aa3cb439-8da3-4fca-ad07-fe00873ec95e"
-					(reference "J16")
+					(reference "J13")
 					(unit 1)
 				)
@@
 		(dnp no)
 		(fields_autoplaced yes)
-		(property "Reference" "J22"
+		(property "Reference" "J8"
 			(at 171.45 107.95 0)
 			(effects
@@
 			(project "modular_software_configurable_io_plc"
 				(path "/b764ffe3-5231-4422-b46d-b0de4c44c7b4/aa3cb439-8da3-4fca-ad07-fe00873ec95e"
-					(reference "J22")
+					(reference "J8")
 					(unit 1)
 				)
@@
 		(dnp no)
 		(fields_autoplaced yes)
-		(property "Reference" "J19"
+		(property "Reference" "J9"
 			(at 151.13 106.68 0)
 			(effects
@@
 			(project "modular_software_configurable_io_plc"
 				(path "/b764ffe3-5231-4422-b46d-b0de4c44c7b4/aa3cb439-8da3-4fca-ad07-fe00873ec95e"
-					(reference "J19")
+					(reference "J9")
 					(unit 1)
 				)
@@
 		(dnp no)
 		(fields_autoplaced yes)
-		(property "Reference" "J18"
+		(property "Reference" "J19"
 			(at 162.56 95.25 0)
 			(effects
@@
 			(project "modular_software_configurable_io_plc"
 				(path "/b764ffe3-5231-4422-b46d-b0de4c44c7b4/aa3cb439-8da3-4fca-ad07-fe00873ec95e"
-					(reference "J18")
+					(reference "J19")
 					(unit 1)
 				)
