File: modular_software_configurable_io_plc/Minimal_LT8304.kicad_sch (KiCad schematic)
At the start: 3 parts, among them J31 CLP-102-02-G-D-BE, J34 CLP-102-02-G-D-BE

Commit message: Backup
Parts:
- renumbered J31 to J1, J34 to J14, MOD8 to MOD3
Changed lines of the file:
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@@
 		(on_board yes)
 		(dnp no)
-		(property "Reference" "J34"
+		(property "Reference" "J14"
 			(at 152.4 88.9 0)
 			(effects
@@
 			(project "modular_software_configurable_io_plc"
 				(path "/b764ffe3-5231-4422-b46d-b0de4c44c7b4/4f7f8433-2347-44be-9a2c-f7cb646575a7"
-					(reference "J34")
+					(reference "J14")
 					(unit 1)
 				)
@@
 		(on_board yes)
 		(dnp no)
-		(property "Reference" "J31"
+		(property "Reference" "J1"
 			(at 128.27 66.04 0)
 			(effects
@@
 			(project "modular_software_configurable_io_plc"
 				(path "/b764ffe3-5231-4422-b46d-b0de4c44c7b4/4f7f8433-2347-44be-9a2c-f7cb646575a7"
-					(reference "J31")
+					(reference "J1")
 					(unit 1)
 				)
@@
 		(dnp no)
 		(fields_autoplaced yes)
-		(property "Reference" "MOD8"
+		(property "Reference" "MOD3"
 			(at 148.59 83.185 0)
 			(effects
@@
 			(project "modular_software_configurable_io_plc"
 				(path "/b764ffe3-5231-4422-b46d-b0de4c44c7b4/4f7f8433-2347-44be-9a2c-f7cb646575a7"
-					(reference "MOD8")
+					(reference "MOD3")
 					(unit 1)
 				)
