File: modular_software_configurable_io_plc/Minimal_LTC9111.kicad_sch (KiCad schematic)
At the start: 5 parts, among them J20 CLP-102-02-G-D-BE, J21 CLP-102-02-G-D-BE, J35 CLP-102-02-G-D-BE, J36 CLP-103-02-G-D-BE

Commit message: Backup
Parts:
- renumbered J35 to J11, J21 to J12, J20 to J37, J36 to J4
Changed lines of the file:
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@@
 		(dnp no)
 		(fields_autoplaced yes)
-		(property "Reference" "J35"
+		(property "Reference" "J11"
 			(at 152.4 91.44 0)
 			(effects
@@
 			(project "modular_software_configurable_io_plc"
 				(path "/b764ffe3-5231-4422-b46d-b0de4c44c7b4/0b69c526-b598-4331-8146-cbb0bf9989e6"
-					(reference "J35")
+					(reference "J11")
 					(unit 1)
 				)
@@
 		(on_board yes)
 		(dnp no)
-		(property "Reference" "J20"
+		(property "Reference" "J37"
 			(at 114.3 80.01 0)
 			(effects
@@
 			(project "modular_software_configurable_io_plc"
 				(path "/b764ffe3-5231-4422-b46d-b0de4c44c7b4/0b69c526-b598-4331-8146-cbb0bf9989e6"
-					(reference "J20")
+					(reference "J37")
 					(unit 1)
 				)
@@
 		(dnp no)
 		(fields_autoplaced yes)
-		(property "Reference" "J21"
+		(property "Reference" "J12"
 			(at 165.1 80.01 0)
 			(effects
@@
 			(project "modular_software_configurable_io_plc"
 				(path "/b764ffe3-5231-4422-b46d-b0de4c44c7b4/0b69c526-b598-4331-8146-cbb0bf9989e6"
-					(reference "J21")
+					(reference "J12")
 					(unit 1)
 				)
@@
 		(dnp no)
 		(fields_autoplaced yes)
-		(property "Reference" "J36"
+		(property "Reference" "J4"
 			(at 133.35 100.33 0)
 			(effects
@@
 			(project "modular_software_configurable_io_plc"
 				(path "/b764ffe3-5231-4422-b46d-b0de4c44c7b4/0b69c526-b598-4331-8146-cbb0bf9989e6"
-					(reference "J36")
+					(reference "J4")
 					(unit 1)
 				)
