File: modular_software_configurable_io_plc/Minimal_MAX14906.kicad_sch (KiCad schematic)
At the start: 9 parts, among them J1 FW-09-03-G-D-085-155, J25 FW-02-03-G-D-085-155, J26 FW-02-03-G-D-085-155, J27 FW-02-03-G-D-085-155, J28 FW-02-03-G-D-085-155, J29 FW-05-03-G-D-085-155, J33 CLP-102-02-G-D-BE, J9 FW-09-03-G-D-085-155

Commit message: Backup
Parts:
- renumbered J29 to J18, J25 to J21, J28 to J22, J26 to J28, J27 to J29, J33 to J34, J9 to J35, J1 to J36, MOD2 to MOD7
Changed lines of the file:
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@@
 		(dnp no)
 		(fields_autoplaced yes)
-		(property "Reference" "J28"
+		(property "Reference" "J22"
 			(at 128.27 127 0)
 			(effects
@@
 			(project "modular_software_configurable_io_plc"
 				(path "/b764ffe3-5231-4422-b46d-b0de4c44c7b4/ef0c2969-c00e-495f-90c1-946f3725c0e6"
-					(reference "J28")
+					(reference "J22")
 					(unit 1)
 				)
@@
 		(dnp no)
 		(fields_autoplaced yes)
-		(property "Reference" "J25"
+		(property "Reference" "J21"
 			(at 168.91 110.49 0)
 			(effects
@@
 			(project "modular_software_configurable_io_plc"
 				(path "/b764ffe3-5231-4422-b46d-b0de4c44c7b4/ef0c2969-c00e-495f-90c1-946f3725c0e6"
-					(reference "J25")
+					(reference "J21")
 					(unit 1)
 				)
@@
 		(dnp no)
 		(fields_autoplaced yes)
-		(property "Reference" "J9"
+		(property "Reference" "J35"
 			(at 118.11 80.0099 90)
 			(effects
@@
 			(project "modular_software_configurable_io_plc"
 				(path "/b764ffe3-5231-4422-b46d-b0de4c44c7b4/ef0c2969-c00e-495f-90c1-946f3725c0e6"
-					(reference "J9")
+					(reference "J35")
 					(unit 1)
 				)
@@
 		(dnp no)
 		(fields_autoplaced yes)
-		(property "Reference" "MOD2"
+		(property "Reference" "MOD7"
 			(at 152.4 118.11 0)
 			(effects
@@
 			(project "modular_software_configurable_io_plc"
 				(path "/b764ffe3-5231-4422-b46d-b0de4c44c7b4/ef0c2969-c00e-495f-90c1-946f3725c0e6"
-					(reference "MOD2")
+					(reference "MOD7")
 					(unit 1)
 				)
@@
 		(dnp no)
 		(fields_autoplaced yes)
-		(property "Reference" "J29"
+		(property "Reference" "J18"
 			(at 168.91 123.19 0)
 			(effects
@@
 			(project "modular_software_configurable_io_plc"
 				(path "/b764ffe3-5231-4422-b46d-b0de4c44c7b4/ef0c2969-c00e-495f-90c1-946f3725c0e6"
-					(reference "J29")
+					(reference "J18")
 					(unit 1)
 				)
@@
 		(dnp no)
 		(fields_autoplaced yes)
-		(property "Reference" "J27"
+		(property "Reference" "J29"
 			(at 168.91 92.71 0)
 			(effects
@@
 			(project "modular_software_configurable_io_plc"
 				(path "/b764ffe3-5231-4422-b46d-b0de4c44c7b4/ef0c2969-c00e-495f-90c1-946f3725c0e6"
-					(reference "J27")
+					(reference "J29")
 					(unit 1)
 				)
@@
 		(dnp no)
 		(fields_autoplaced yes)
-		(property "Reference" "J33"
+		(property "Reference" "J34"
 			(at 115.57 109.22 0)
 			(effects
@@
 			(project "modular_software_configurable_io_plc"
 				(path "/b764ffe3-5231-4422-b46d-b0de4c44c7b4/ef0c2969-c00e-495f-90c1-946f3725c0e6"
-					(reference "J33")
+					(reference "J34")
 					(unit 1)
 				)
@@
 		(dnp no)
 		(fields_autoplaced yes)
-		(property "Reference" "J26"
+		(property "Reference" "J28"
 			(at 129.54 93.98 0)
 			(effects
@@
 			(project "modular_software_configurable_io_plc"
 				(path "/b764ffe3-5231-4422-b46d-b0de4c44c7b4/ef0c2969-c00e-495f-90c1-946f3725c0e6"
-					(reference "J26")
+					(reference "J28")
 					(unit 1)
 				)
@@
 		(dnp no)
 		(fields_autoplaced yes)
-		(property "Reference" "J1"
+		(property "Reference" "J36"
 			(at 176.53 80.0099 90)
 			(effects
@@
 			(project "modular_software_configurable_io_plc"
 				(path "/b764ffe3-5231-4422-b46d-b0de4c44c7b4/ef0c2969-c00e-495f-90c1-946f3725c0e6"
-					(reference "J1")
+					(reference "J36")
 					(unit 1)
 				)
